Commit message: add fake hardware args

File: urdf/pick_place.xacro (robot description, xacro)
@@ -1,4 +1,7 @@
 <?xml version="1.0"?>
 <robot name="gen3_2f_85_pick_place" xmlns:xacro="http://ros.org/wiki/xacro">
+  <!-- arguments -->
+  <xacro:arg name="use_fake_hardware" default="false" />
+  <xacro:arg name="fake_sensor_commands" default="false" />
   <xacro:property name="PI" value="3.14159265359" />
   <xacro:property name="prefix" value="kinova_" />
@@ -7,5 +10,5 @@
   <xacro:property name="dof" value="7" />
   <xacro:property name="gripper" value="robotiq_2f_85" />
-  <xacro:property name="gripper_joint_name" default="finger_joint" />
+  <xacro:property name="gripper_joint_name" default="" />
   <xacro:property name="robot_ip" default="192.168.0.11" />
   <xacro:property name="username" default="admin" />
@@ -80,4 +83,6 @@
     parent="${prefix}table_mount"
     vision="true"
+    use_fake_hardware="$(arg use_fake_hardware)"
+    fake_sensor_commands="$(arg fake_sensor_commands)"
     robot_ip="${robot_ip}"
     username="${username}"

Commit message: add bringup launch file and some fixes

File: urdf/pick_place.xacro (robot description, xacro)
@@ -4,4 +4,6 @@
   <xacro:arg name="use_fake_hardware" default="false" />
   <xacro:arg name="fake_sensor_commands" default="false" />
+  <xacro:arg name="robot_ip" default="" />
+  <xacro:arg name="gripper_joint_name" default="" />
   <xacro:property name="PI" value="3.14159265359" />
   <xacro:property name="prefix" value="kinova_" />
@@ -10,6 +12,4 @@
   <xacro:property name="dof" value="7" />
   <xacro:property name="gripper" value="robotiq_2f_85" />
-  <xacro:property name="gripper_joint_name" default="" />
-  <xacro:property name="robot_ip" default="192.168.0.11" />
   <xacro:property name="username" default="admin" />
   <xacro:property name="password" default="admin" />
@@ -85,5 +85,5 @@
     use_fake_hardware="$(arg use_fake_hardware)"
     fake_sensor_commands="$(arg fake_sensor_commands)"
-    robot_ip="${robot_ip}"
+    robot_ip="$(arg robot_ip)"
     username="${username}"
     password="${password}"
@@ -92,5 +92,6 @@
     session_inactivity_timeout_ms="${session_inactivity_timeout_ms}"
     connection_inactivity_timeout_ms="${connection_inactivity_timeout_ms}"
-    gripper_joint_name="${gripper_joint_name}">
+    gripper_joint_name="$(arg gripper_joint_name)"
+    use_internal_bus_gripper_comm="true">
     <origin xyz="0 0 ${0.026/2}" rpy="0 0 ${robot_origin_yaw}"/>
   </xacro:load_robot>

Commit message: PC clustering, detection of cubes and spheres xacro fixes launch file param fixes sort_objects node refractor

File: urdf/pick_place.xacro (robot description, xacro)
@@ -6,6 +6,6 @@
   <xacro:arg name="robot_ip" default="" />
   <xacro:arg name="gripper_joint_name" default="" />
+  <xacro:arg name="prefix" default="" />
   <xacro:property name="PI" value="3.14159265359" />
-  <xacro:property name="prefix" value="kinova_" />
   <!-- parameters -->
   <xacro:property name="arm" value="gen3" />
@@ -48,5 +48,5 @@
   </xacro:table>
   <!-- kinova table mount -->
-  <link name="${prefix}table_mount">
+  <link name="$(arg prefix)table_mount">
     <visual>
       <origin xyz="0 0 0" rpy="0 0 0"/>
@@ -70,7 +70,7 @@
   <xacro:property name="mount_origin_z" value="0.013" />
   <xacro:property name="robot_origin_yaw" value="${PI/2}" />
-  <joint name="${prefix}table_mount_joint" type="fixed">
+  <joint name="$(arg prefix)table_mount_joint" type="fixed">
     <parent link="${table_prefix}_top"/>
-    <child link="${prefix}table_mount"/>
+    <child link="$(arg prefix)table_mount"/>
     <origin xyz="${mount_origin_x} ${mount_origin_y} ${mount_origin_z}" rpy="0 0 0"/>
   </joint>
@@ -80,6 +80,6 @@
     dof="${dof}"
     gripper="${gripper}"
-    prefix="${prefix}"
-    parent="${prefix}table_mount"
+    prefix="$(arg prefix)"
+    parent="$(arg prefix)table_mount"
     vision="true"
     use_fake_hardware="$(arg use_fake_hardware)"
@@ -100,8 +100,8 @@
   <xacro:property name="robotiq_85_base_tip_closed_length" value="0.1628" />
   <!-- robotiq 2f-85 grasp link -->
-  <link name="${prefix}robotiq_85_grasp_link" />
-  <joint name="${prefix}robotiq_85_grasp_joint" type="fixed">
-    <parent link="${prefix}robotiq_85_base_link"/>
-    <child link="${prefix}robotiq_85_grasp_link"/>
+  <link name="$(arg prefix)robotiq_85_grasp_link" />
+  <joint name="$(arg prefix)robotiq_85_grasp_joint" type="fixed">
+    <parent link="$(arg prefix)robotiq_85_base_link"/>
+    <child link="$(arg prefix)robotiq_85_grasp_link"/>
     <origin rpy="0 0 0" xyz="0 0 ${robotiq_85_base_tip_open_length}"/>
   </joint>

Commit message: some fixes i think

File: urdf/pick_place.xacro (robot description, xacro)
@@ -6,5 +6,5 @@
   <xacro:arg name="robot_ip" default="" />
   <xacro:arg name="gripper_joint_name" default="" />
-  <xacro:arg name="prefix" default="" />
+  <xacro:arg name="prefix" default="kinova_" />
   <xacro:property name="PI" value="3.14159265359" />
   <!-- parameters -->
@@ -35,4 +35,30 @@
   <!-- world -->
   <link name="world"/>
+  <xacro:property name="wall_height" value="2.0" />
+  <xacro:property name="wall_Y_offset" value="${table_top_breadth/2 + (table_leg_breadth/2)}" />
+  <xacro:property name="wall_Y" value="${wall_Y_offset + 0.3 - 0.025}" />
+  <!-- wall -->
+  <link name="wall">
+    <visual>
+      <origin xyz="0 ${-wall_Y} ${wall_height/2} " rpy="0 0 0"/>
+      <geometry>
+        <box size="${wall_height*1.5} 0.05 ${wall_height}"/>
+      </geometry>
+      <material name="not_white">
+        <color rgba="0.7 0.7 0.7 1.0"/>
+      </material>
+    </visual>
+    <collision>
+      <origin xyz="0 ${-wall_Y} ${wall_height/2} " rpy="0 0 0"/>
+      <geometry>
+        <box size="${wall_height*1.5} 0.05 ${wall_height}"/>
+      </geometry>
+    </collision>
+  </link>
+  <joint name="wall_joint" type="fixed">
+    <parent link="world"/>
+    <child link="wall"/>
+    <origin xyz="0 0 0" rpy="0 0 0"/>
+  </joint>
   <!-- table -->
   <xacro:table prefix="${table_prefix}"
